File: kicad/25v-Supply.kicad_sch (KiCad schematic)
At the start: 16 parts, among them IC1 NE555P, T1 22uf, T2 22uf, T3 2.2uf, T4 2.2uf

Commit message: Kicad 9 and Docs
Parts:
- D1, D2: footprint Diode_THT:D_DO-41_SOD81_P12.70mm_Horizontal -> Diode_THT:D_DO-35_SOD27_P12.70mm_Horizontal
